File: 5V 3V3.kicad_sch (KiCad schematic)
At the start: 27 parts, among them U1 SY7088DGC, U2 DRV8833PWP, U3 AP2114H-3.3TRG1, U5 RT9742GGJ5

Commit message: final upload of wtv with feet
Parts:
- removed C13: 10nF, C0402, symbol Component Importer-altium-import:root_0_CL05B103KB5NNNC_
- removed C14: 22uF, C1206, symbol Component Importer-altium-import:root_0_CL31A226KAHNNNE_
- removed C15, C5: 1uF, C0603, symbol Component Importer-altium-import:root_0_CL10A105KB8NNNC_
- removed C2: 2.2uF, C0402, symbol Component Importer-altium-import:root_0_CL05A225MQ5NSNC_
- removed C8: 10uF, C0805, symbol Component Importer-altium-import:root_0_CL21A106KAYNNNE_C15850_
- removed L1: 1.5uH, IND-SMD_L4.0-W4.0, symbol Component Importer-altium-import:root_0_SWPA4020S1R5NT_
- removed R2, R4: R_Small_US, symbol Device:R_Small_US
- removed R3: 10kΩ, R0603, symbol Component Importer-altium-import:root_0_0603WAF1002T5E_
- removed R6: 1MΩ, R0805, symbol Component Importer-altium-import:root_0_0805W8F1004T5E_
- removed U3: AP2114H-3.3TRG1, SOT-223_L6.7-W3.5-P2.30-BR, symbol Component Importer-altium-import:root_0_AP2114H-3.3TRG1_
- removed U5: RT9742GGJ5, TSOT-23-5_L2.9-W1.6-P0.95-LS2.8-BR, symbol Component Importer-altium-import:root_0_RT9742GGJ5_
- added C11: 10nF, Capacitor_SMD:C_0402_1005Metric_Pad0.74x0.62mm_HandSolder, symbol Component Importer-altium-import:root_0_CL05B103KB5NNNC_
- added C13: 2.2uF, Capacitor_SMD:C_0402_1005Metric_Pad0.74x0.62mm_HandSolder, symbol Component Importer-altium-import:root_0_CL05A225MQ5NSNC_
- added C16, C18: 1uF, Capacitor_SMD:C_0603_1608Metric_Pad1.08x0.95mm_HandSolder, symbol Component Importer-altium-import:root_0_CL10A105KB8NNNC_
- added C17: 10uF, Capacitor_SMD:C_0805_2012Metric_Pad1.18x1.45mm_HandSolder, symbol Component Importer-altium-import:root_0_CL21A106KAYNNNE_C15850_
- added C2: 22uF, Capacitor_SMD:C_1206_3216Metric_Pad1.33x1.80mm_HandSolder, symbol Component Importer-altium-import:root_0_CL31A226KAHNNNE_
- added IC1: AP2114H-3.3TRG1, Library:SOT-223_L6.7-W3.5-P2.30-BR, symbol AP2114H-3.3TRG1:AP2114H-3.3TRG1
- added L1: SWPA4020S1R5NT, Inductor_SMD:L_Cenker_CKCS4018, symbol Device:L
- added R10, R11, R12: 1Ω, Resistor_SMD:R_1206_3216Metric_Pad1.30x1.75mm_HandSolder, symbol Component Importer-altium-import:root_0_1206W4F100KT5E_
- added R2: 1MΩ, Resistor_SMD:R_0805_2012Metric_Pad1.20x1.40mm_HandSolder, symbol Component Importer-altium-import:root_0_0805W8F1004T5E_
- added R8, R9: 10kΩ, Resistor_SMD:R_0603_1608Metric_Pad0.98x0.95mm_HandSolder, symbol Component Importer-altium-import:root_0_0603WAF1002T5E_
- added SW1: SS-12D11G3R, Library:SW-TH_SS-12D11L3, symbol Component Importer-altium-import:root_0_SS-12D11G3R_
- added TP0, TP1, TP2, TP3, TP4, TP5: TestPoint, TestPoint:TestPoint_Pad_D3.0mm, symbol Connector:TestPoint
- added U5, U6: RT9742GGJ5, Package_TO_SOT_SMD:TSOT-23-5, symbol RT9742GGJ5:RT9742GGJ5
- C1: footprint C1206 -> Capacitor_SMD:C_1206_3216Metric_Pad1.33x1.80mm_HandSolder; LCSC (none) -> C12891
- C10: footprint C0402 -> Capacitor_SMD:C_0402_1005Metric_Pad0.74x0.62mm_HandSolder; LCSC (none) -> C15195
- C12: footprint C0805 -> Capacitor_SMD:C_0805_2012Metric_Pad1.18x1.45mm_HandSolder; LCSC (none) -> C15850
- C3, C4: footprint C0603 -> Capacitor_SMD:C_0603_1608Metric_Pad1.08x0.95mm_HandSolder; LCSC (none) -> C19666
- C6: footprint C0603 -> Capacitor_SMD:C_0603_1608Metric_Pad1.08x0.95mm_HandSolder; LCSC (none) -> C15849
- C7: footprint C0402 -> Capacitor_SMD:C_0402_1005Metric_Pad0.74x0.62mm_HandSolder; LCSC (none) -> C12530
- C9: footprint C1206 -> Capacitor_SMD:C_1206_3216Metric_Pad1.33x1.80mm_HandSolder; LCSC (none) -> C15008
- R1: footprint R0805 -> Resistor_SMD:R_0805_2012Metric_Pad1.20x1.40mm_HandSolder; LCSC (none) -> C17514
- R5: footprint R0603 -> Resistor_SMD:R_0603_1608Metric_Pad0.98x0.95mm_HandSolder; LCSC (none) -> C25804
- R7: footprint R0603 -> Resistor_SMD:R_0603_1608Metric_Pad0.98x0.95mm_HandSolder; LCSC (none) -> C23137
- U1: footprint DFN-8_L3.0-W2.0-P0.50-BL-EP -> Library:DFN-8_L3.0-W2.0-P0.50-BL-EP; LCSC (none) -> C178240
- U2: LCSC (none) -> C1556089
- U4: renamed from U?; LCSC (none) -> C1556089
Connections:
- net GND: now also C13.1, C16.1, C17.2, C18.1, C2.1, IC1.1 (GND), R10.1, R11.1, R12.1, R8.2, TP1.1, TP3.1, TP4.1, U5.P$2 (GND), U6.P$2 (GND)
- net Battery: now reaches C12.1, U2.12 (VM)
- net Battery: now also C1.2, C10.1, C3.2, C9.2, R1.2, R5.1, U1.3 (EN), U1.6 (IN), U4.12 (VM), C11.1, C17.1, C18.2, IC1.3 (VIN), L1.1, R9.1, SW1.1
- net 5V Out: now reaches C6.2
- net 5V Out: now also U1.8 (OUT), C16.2, C2.2, R2.2, U5.P$5 (IN), U6.P$5 (IN)
- net at U2.3 (AISEN), U2.6 (BISEN): now also R12.2, TP0.1
- net at U4.1 (~{SLEEP}): now also R9.2
- net MOTOR4_CTRL2: now reaches U4.10 (BIN2)
- net at U4.11 (VCP): now also C11.2
- net MOTOR3_CTRL2: now reaches U4.15 (AIN2)
- net MOTOR3_CTRL1: now reaches U4.16 (AIN1)
- net MOTOR3_A_OUT: now reaches U4.2 (AOUT1)
- net at U4.3 (AISEN), U4.6 (BISEN): now also R10.2, R11.2, TP2.1
- net MOTOR3_B_OUT: now reaches U4.4 (AOUT2)
- net Motor4_B_OUT: now reaches U4.5 (BOUT2)
- net Motor4_A_OUT: now reaches U4.7 (BOUT1)
- net MOTOR4_CTRL1: now reaches U4.9 (BIN1)
- net 3V3 Out: now reaches C4.2
- net 3V3 Out: now also IC1.2 (VOUT_1)
- net MOTOR2_CTRL2: now reaches U2.10 (BIN2)
- net at U2.14 (VINT): now also C13.2
- net MOTOR1_CTRL2: now reaches U2.15 (AIN2)
- net MOTOR1_CTRL1: now reaches U2.16 (AIN1)
- net MOTOR1_A_OUT: now reaches U2.2 (AOUT1)
- net MOTOR1_B_OUT: now reaches U2.4 (AOUT2)
- net Motor2_B_OUT: now reaches U2.5 (BOUT2)
- net Motor2_A_OUT: now reaches U2.7 (BOUT1)
- net MOTOR2_CTRL1: now reaches U2.9 (BIN1)
- net at U1.1 (LX): now also L1.2
- net at R7.2, U1.5 (FB): now also R2.1
- new net: R8.1, SW1.3, TP5.1
- new net CTRL_EXT_LOAD1: U5.P$4 (EN)
- new net CTRL_EXT_LOAD2: U6.P$4 (EN)
- new net EXT_LOAD1_OUT: U5.P$1 (OUT)
- new net EXT_LOAD2_OUT: U6.P$1 (OUT)
- new net Slider switch: SW1.2
- no-connect marks 0 -> 8
Other:
- note added: "3V3 OUT @300mA MAX"
- note added: "5V OUT @1.5A MAX"
- note added: "Auxiliary motors @500mA"
- note added: "Control motors @200mA"
- note added: "External load switching at 1A"
- note added: "ON/OFF switch"
- moved on the sheet: C10, C12, C3, C6, C7, R5, U4
