File: Power_Board_v2/Power_Board_v2.kicad_sch (KiCad schematic)
At the start: 34 parts, among them J1 PH2.54-01-16PZS, J2 Conn_01x02, Q1 MMBT5551L, U2 HUSB237-AA001-DN06R, U3 BQ24074RGT, U4 INA219AIDCNR

Commit message: yes 3
Parts:
- added C1, C2: 22uF, Capacitor_SMD:C_1206_3216Metric_Pad1.33x1.80mm_HandSolder, symbol Component Importer-altium-import:root_0_CL31A226KAHNNNE_
- added C10, C16, C18: 1uF, Capacitor_SMD:C_0603_1608Metric_Pad1.08x0.95mm_HandSolder, symbol Component Importer-altium-import:root_0_CL10A105KB8NNNC_
- added C11, C3: 4.7uF, Capacitor_SMD:C_0603_1608Metric_Pad1.08x0.95mm_HandSolder, symbol Component Importer-altium-import:root_0_CL10A475KO8NNNC_
- added C12, C13: 10nF, Capacitor_SMD:C_0402_1005Metric_Pad0.74x0.62mm_HandSolder, symbol Component Importer-altium-import:root_0_CL05B103KB5NNNC_
- added C14, C15: 2.2uF, Capacitor_SMD:C_0402_1005Metric_Pad0.74x0.62mm_HandSolder, symbol Component Importer-altium-import:root_0_CL05A225MQ5NSNC_
- added C17, C19: 10uF, Capacitor_SMD:C_0805_2012Metric_Pad1.18x1.45mm_HandSolder, symbol Component Importer-altium-import:root_0_CL21A106KAYNNNE_C15850_
- added C9: 100uF, Capacitor_SMD:C_1206_3216Metric_Pad1.33x1.80mm_HandSolder, symbol Component Importer-altium-import:root_0_CL31A107MQHNNNE_
- added IC1: AP2114H-3.3TRG1, Library:SOT-223_L6.7-W3.5-P2.30-BR, symbol AP2114H-3.3TRG1:AP2114H-3.3TRG1
- added L1: SWPA4020S1R5NT, Inductor_SMD:L_Cenker_CKCS4018, symbol Device:L
- added R1, R5: 1MΩ, Resistor_SMD:R_0805_2012Metric_Pad1.20x1.40mm_HandSolder, symbol Component Importer-altium-import:root_0_0805W8F1004T5E_
- added R19, R23, R6: 10kΩ, Resistor_SMD:R_0603_1608Metric_Pad0.98x0.95mm_HandSolder, symbol Component Importer-altium-import:root_0_0603WAF1002T5E_
- added R20, R21, R22: 1Ω, Resistor_SMD:R_1206_3216Metric_Pad1.30x1.75mm_HandSolder, symbol Component Importer-altium-import:root_0_1206W4F100KT5E_
- added R8: 330kΩ, Resistor_SMD:R_0603_1608Metric_Pad0.98x0.95mm_HandSolder, symbol Component Importer-altium-import:root_0_0603WAF3303T5E_
- added SW1: SS-12D11G3R, Library:SW-TH_SS-12D11L3, symbol Component Importer-altium-import:root_0_SS-12D11G3R_
- added TP10, TP11, TP12, TP7, TP8, TP9: TestPoint, TestPoint:TestPoint_Pad_D3.0mm, symbol Connector:TestPoint
- added U1: SY7088DGC, Library:DFN-8_L3.0-W2.0-P0.50-BL-EP, symbol Component Importer-altium-import:root_0_SY7088DGC_
- added U5, U6: RT9742GGJ5, Package_TO_SOT_SMD:TSOT-23-5, symbol RT9742GGJ5:RT9742GGJ5
- added U7, U8: DRV8833PWP, Package_SO:HTSSOP-16-1EP_4.4x5mm_P0.65mm_EP3.4x5mm_Mask2.46x2.31mm_ThermalVias, symbol Driver_Motor:DRV8833PWP
Connections:
- net 3V3 Out: now also C11.2, IC1.2 (VOUT_1)
- net 5V Out: now also C10.2, C16.2, C2.2, R5.2, U1.8 (OUT), U5.P$5 (IN), U6.P$5 (IN)
- net Battery: now also C1.2, C12.1, C13.1, C17.1, C18.2, C19.1, C3.2, C9.2, IC1.3 (VIN), L1.1, R1.2, R23.1, R6.1, SW1.1, U1.3 (EN), U1.6 (IN), U7.12 (VM), U8.12 (VM)
- net CTRL_EXT_LOAD1: now also U5.P$4 (EN)
- net CTRL_EXT_LOAD2: now also U6.P$4 (EN)
- net EXT_LOAD1_OUT: now also U5.P$1 (OUT)
- net EXT_LOAD2_OUT: now also U6.P$1 (OUT)
- net GND: now also C1.1, C10.1, C11.1, C14.1, C15.1, C16.1, C17.2, C18.1, C19.2, C2.1, C3.1, C9.1, IC1.1 (GND), R1.1, R19.2, R20.1, R21.1, R22.1, R8.1, TP10.1, TP12.1, TP8.1, U1.9 (PGND), U5.P$2 (GND), U6.P$2 (GND), U7.13 (GND), U7.17 (GND), U8.13 (GND), U8.17 (GND)
- net MOTOR1_A_OUT: now also U7.2 (AOUT1)
- net MOTOR1_B_OUT: now also U7.4 (AOUT2)
- net MOTOR1_CTRL1: now also U7.16 (AIN1)
- net MOTOR1_CTRL2: now also U7.15 (AIN2)
- net MOTOR2_CTRL1: now also U7.9 (BIN1)
- net MOTOR2_CTRL2: now also U7.10 (BIN2)
- net MOTOR3_A_OUT: now also U8.2 (AOUT1)
- net MOTOR3_B_OUT: now also U8.4 (AOUT2)
- net MOTOR3_CTRL1: now also U8.16 (AIN1)
- net MOTOR3_CTRL2: now also U8.15 (AIN2)
- net MOTOR4_CTRL1: now also U8.9 (BIN1)
- net MOTOR4_CTRL2: now also U8.10 (BIN2)
- net Motor2_A_OUT: now also U7.7 (BOUT1)
- net Motor2_B_OUT: now also U7.5 (BOUT2)
- net Motor4_A_OUT: now also U8.7 (BOUT1)
- net Motor4_B_OUT: now also U8.5 (BOUT2)
- new net: R5.1, R8.2, U1.5 (FB)
- new net: C14.2, U7.14 (VINT)
- new net: R23.2, U8.1 (~{SLEEP})
- new net: C13.2, U8.11 (VCP)
- new net: C15.2, U8.14 (VINT)
- new net: R20.2, R22.2, TP9.1, U8.3 (AISEN), U8.6 (BISEN)
- new net: R6.2, U7.1 (~{SLEEP})
- new net: C12.2, U7.11 (VCP)
- new net: R21.2, TP11.1, U7.3 (AISEN), U7.6 (BISEN)
- new net: L1.2, U1.1 (LX)
- new net: R19.1, SW1.3, TP7.1
- new net Slider switch: SW1.2
- no-connect marks 14 -> 22
Other:
- note added: "3V3 OUT @300mA MAX"
- note added: "5V OUT @1.5A MAX"
- note added: "Auxiliary motors @500mA"
- note added: "Control motors @200mA"
- note added: "External load switching at 1A"
- note added: "ON/OFF switch"
- note added: "YES"

Commit message: idek
Parts:
- IC1: footprint Library:SOT-223_L6.7-W3.5-P2.30-BR -> libbypretty:SOT-223_L6.7-W3.5-P2.30-BR
- SW1: footprint Library:SW-TH_SS-12D11L3 -> libbypretty:SW-TH_SS-12D11L3
- U1: footprint Library:DFN-8_L3.0-W2.0-P0.50-BL-EP -> libbypretty:DFN-8_L3.0-W2.0-P0.50-BL-EP
Changed lines of the file:
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@@
 			)
 		)
-		(property "Footprint" "Library:DFN-8_L3.0-W2.0-P0.50-BL-EP"
+		(property "Footprint" "libbypretty:DFN-8_L3.0-W2.0-P0.50-BL-EP"
 			(at 66.04 226.06 0)
 			(effects
@@
 			)
 		)
-		(property "Footprint" "Library:SW-TH_SS-12D11L3"
+		(property "Footprint" "libbypretty:SW-TH_SS-12D11L3"
 			(at 180.34 167.64 0)
 			(effects
@@
 			)
 		)
-		(property "Footprint" "Library:SOT-223_L6.7-W3.5-P2.30-BR"
+		(property "Footprint" "libbypretty:SOT-223_L6.7-W3.5-P2.30-BR"
 			(at 219.71 224.79 0)
 			(effects
