File: Power_Board_v2/Power_Board_v2.kicad_pcb (KiCad board)
At the start: 2 copper layers, 68 parts, among them J1 PH2.54-01-16PZS, J2 Conn_01x02, Q1 MMBT5551L, U2 HUSB237-AA001-DN06R, U3 BQ24074RGT, U4 INA219AIDCNR, U5 RT9742GGJ5, U6 RT9742GGJ5, U7 DRV8833PWP, U8 DRV8833PWP

Commit message: Connected up the last passive stuff
Parts:
- moved C10 78.6 mm to (222.0, 141.0), turned to 0 degrees
- moved C11 59.6 mm to (207.1, 133.0), turned to 0 degrees
- moved C3 51.1 mm to (196.0, 117.9)
- moved R6 46.6 mm to (204.0, 113.0), turned to 0 degrees
- moved C18 43.1 mm to (198.0, 113.0), turned to 0 degrees
Routing:
- net /Battery: track 292.5 -> 321.7 mm
- net Net-(U7-~{SLEEP}): track 0.00 -> 8.84 mm
- net /5V Out: track 68.9 -> 73.5 mm
